File: projects/actuatorboard/actuatorboard.brd (EAGLE design)
At the start: 87 x 55 mm, 67 parts, among them P1 39-30-04?

Commit message: Fixed board outline on actuator board.
Parts:
- PCB1: value BEAGLEBONE_BLACK_CAPE -> BEAGLEBONE_BLACK_CAPENO_ETH; device e14_BeagleBoneBlack_RevB:BEAGLEBONE_BLACK_CAPE -> e14_BeagleBoneBlack_RevB:BEAGLEBONE_BLACK_CAPE_NO_ETH
Other:
- board size 87 x 55 mm -> 86.4 x 54.6 mm
Changed lines of the file:
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@@
 <?xml version="1.0" encoding="utf-8"?>
 <!DOCTYPE eagle SYSTEM "eagle.dtd">
-<eagle version="7.6.0">
+<eagle version="7.4.0">
 <drawing>
 <settings>
@@
 <board>
 <plain>
-<wire x1="0" y1="0" x2="87" y2="0" width="0" layer="20"/>
-<wire x1="87" y1="0" x2="87" y2="55" width="0" layer="20"/>
-<wire x1="87" y1="55" x2="0" y2="55" width="0" layer="20"/>
-<wire x1="0" y1="55" x2="0" y2="0" width="0" layer="20"/>
 </plain>
 <attributes>
@@
 <element name="U$4" library="transistor" package="SOT363-INFINION" value="BC847PN" x="-12.64" y="36.16"/>
 <element name="LOGO" library="components" package="SU_LOGO_DS" value="SU_LOGO-DUMMY" x="-87.33" y="27.6"/>
-<element name="PCB1" library="e14_BeagleBoneBlack_RevB" package="BEAGLEBONE_BLACK_CAPE" value="BEAGLEBONE_BLACK_CAPE" x="0" y="0"/>
+<element name="PCB1" library="e14_BeagleBoneBlack_RevB" package="BEAGLEBONE_BLACK_CAPE_NO_ETH" value="BEAGLEBONE_BLACK_CAPENO_ETH" x="0" y="0"/>
 <element name="R13" library="rcl" package="R0805" value="10K" x="-16.77" y="39.96"/>
 <element name="D2" library="diode" package="SOT23" value="BAT54S" x="-33.5" y="43.34"/>

Commit message: Actuator board
lotta work done on actuator board
Parts:
- moved LOGO 168.5 mm to (81.2, 23.6)
- moved JMP1 133.0 mm to (55.0, 9.00)
- moved R10 132.0 mm to (59.0, 8.50), turned to 90 degrees
- moved RN7 123.5 mm to (50.5, 8.00), turned to 180 degrees
- moved U$15 116.1 mm to (51.2, 40.8)
- moved RN2 106.7 mm to (31.1, 37.8), turned to 90 degrees
- moved RN3 105.5 mm to (31.1, 29.3), turned to 90 degrees
- moved R4 104.1 mm to (63.6, 12.8)
- moved R14 103.8 mm to (77.7, 13.1), turned to 270 degrees
- moved LED1 103.7 mm to (75.6, 8.40), turned to 180 degrees
- moved D2 103.6 mm to (69.0, 28.3)
- moved R9 103.1 mm to (74.0, 12.9), turned to 90 degrees
- moved U$7 102.2 mm to (60.7, 36.5), turned to 270 degrees
- moved U$11 102.1 mm to (38.5, 41.2), turned to 90 degrees
- moved U$24 101.5 mm to (24.5, 41.9), turned to 270 degrees
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Connections:
- removed net N$91: RN6.1, U$23.16
- new net N$36: RN6.2, U$23.12
- net N$15: now also RN1.4; no longer RN1.1
- net N$16: now also RN2.4; no longer RN2.1
- net N$17: now also RN2.5; no longer RN2.8
- net N$24: now also RN1.3; no longer RN1.2
- net N$25: now also RN2.6; no longer RN2.7
- net N$26: now also RN2.3; no longer RN2.2
- net N$28: now also RN1.2; no longer RN1.3
- net N$29: now also RN2.7; no longer RN2.6
- net N$30: now also RN2.2; no longer RN2.3
- net N$32: now also RN1.1; no longer RN1.4
- net N$33: now also RN2.8; no longer RN2.5
- net N$34: now also RN2.1; no longer RN2.4
- net N$39: now also RN3.5; no longer RN3.8
- net N$40: now also RN3.4; no longer RN3.1
- net N$43: now also RN3.6; no longer RN3.7
- net N$44: now also RN3.3; no longer RN3.2
- net N$47: now also RN3.7; no longer RN3.6
- net N$48: now also RN3.2; no longer RN3.3
- net N$51: now also RN3.8; no longer RN3.5
- net N$52: now also RN3.1; no longer RN3.4
- net N$55: now also RN6.5; no longer RN6.8
- net N$62: now also RN6.6; no longer RN6.7
- net N$63: now also RN6.7; no longer RN6.6
- net N$64: now also RN6.8; no longer RN6.5
- net N$65: now also RN8.5; no longer RN8.8
- net N$70: now also RN8.6; no longer RN8.7
- net N$71: now also RN8.7; no longer RN8.6
- net N$72: now also RN8.8; no longer RN8.5
- net N$78: now also RN8.1; no longer RN8.4
- net N$85: now also RN8.2; no longer RN8.3
- net N$86: now also RN8.3; no longer RN8.2
- net N$87: now also RN8.4; no longer RN8.1
- net N$88: now also RN6.1; no longer RN6.4
- net N$89: now also U$23.14; no longer U$23.12
- net N$90: now also RN6.4, U$23.16; no longer RN6.2, U$23.14
Routing:
- net +12V: track 0.00 -> 106.3 mm, vias 0 -> 8
- net +5V: track 0.00 -> 95.6 mm, vias 0 -> 7
- net +3V3: track 0.00 -> 91.3 mm, vias 0 -> 8
- net !RESET!: track 0.00 -> 47.7 mm, vias 0 -> 6
- net N$2: track 0.00 -> 46.4 mm, vias 0 -> 4
- net N$74: track 0.00 -> 44.9 mm, vias 0 -> 4
- net N$69: track 0.00 -> 44.6 mm, vias 0 -> 4
- net N$72: track 0.00 -> 41.9 mm
- net SCL: track 0.00 -> 40.8 mm, vias 0 -> 4
- net N$68: track 0.00 -> 40.6 mm, vias 0 -> 2
- net SDA: track 0.00 -> 40.0 mm, vias 0 -> 3
- net N$71: track 0.00 -> 39.4 mm
- net N$82: track 0.00 -> 38.5 mm, vias 0 -> 2
- net N$70: track 0.00 -> 36.5 mm
- net N$79: track 0.00 -> 35.8 mm, vias 0 -> 2
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- added copper zone on layer 1, net N$12
