File: projects/actuatorboard/actuatorboard.sch (EAGLE design)
At the start: 67 parts, among them P1 39-30-04

Commit message: Fixed board outline on actuator board.
Parts:
- PCB1: value BEAGLEBONE_BLACK_CAPE -> BEAGLEBONE_BLACK_CAPENO_ETH; device e14_BeagleBoneBlack_RevB:BEAGLEBONE_BLACK_CAPE -> e14_BeagleBoneBlack_RevB:BEAGLEBONE_BLACK_CAPENO_ETH
Changed lines of the file:
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@@
 <part name="LOGO" library="components" deviceset="SU_LOGO-DUMMY" device=""/>
 <part name="GND14" library="supply1" deviceset="GND" device=""/>
-<part name="PCB1" library="e14_BeagleBoneBlack_RevB" deviceset="BEAGLEBONE_BLACK_CAPE" device=""/>
+<part name="PCB1" library="e14_BeagleBoneBlack_RevB" deviceset="BEAGLEBONE_BLACK_CAPE" device="NO_ETH"/>
 <part name="R13" library="rcl" deviceset="R-EU_" device="R0805" value="10K"/>
 <part name="D2" library="diode" deviceset="BAT54S" device=""/>

Commit message: Actuator board
lotta work done on actuator board
Connections:
- removed net N$91: RN6A.1, U$23-16.K
- new net N$36: RN6B.1, U$23-12.K
- net N$15: now also RN1D.1; no longer RN1A.1
- net N$16: now also RN2D.1; no longer RN2A.1
- net N$17: now also RN2D.2; no longer RN2A.2
- net N$24: now also RN1C.1; no longer RN1B.1
- net N$25: now also RN2C.2; no longer RN2B.2
- net N$26: now also RN2C.1; no longer RN2B.1
- net N$28: now also RN1B.1; no longer RN1C.1
- net N$29: now also RN2B.2; no longer RN2C.2
- net N$30: now also RN2B.1; no longer RN2C.1
- net N$32: now also RN1A.1; no longer RN1D.1
- net N$33: now also RN2A.2; no longer RN2D.2
- net N$34: now also RN2A.1; no longer RN2D.1
- net N$39: now also RN3D.2; no longer RN3A.2
- net N$40: now also RN3D.1; no longer RN3A.1
- net N$43: now also RN3C.2; no longer RN3B.2
- net N$44: now also RN3C.1; no longer RN3B.1
- net N$47: now also RN3B.2; no longer RN3C.2
- net N$48: now also RN3B.1; no longer RN3C.1
- net N$51: now also RN3A.2; no longer RN3D.2
- net N$52: now also RN3A.1; no longer RN3D.1
- net N$55: now also RN6D.2; no longer RN6A.2
- net N$62: now also RN6C.2; no longer RN6B.2
- net N$63: now also RN6B.2; no longer RN6C.2
- net N$64: now also RN6A.2; no longer RN6D.2
- net N$65: now also RN8D.2; no longer RN8A.2
- net N$70: now also RN8C.2; no longer RN8B.2
- net N$71: now also RN8B.2; no longer RN8C.2
- net N$72: now also RN8A.2; no longer RN8D.2
- net N$78: now also RN8A.1; no longer RN8D.1
- net N$85: now also RN8B.1; no longer RN8C.1
- net N$86: now also RN8C.1; no longer RN8B.1
- net N$87: now also RN8D.1; no longer RN8A.1
- net N$88: now also RN6A.1; no longer RN6D.1
- net N$89: now also U$23-14.K; no longer U$23-12.K
- net N$90: now also RN6D.1, U$23-16.K; no longer RN6B.1, U$23-14.K
Other:
- moved on the sheet: RN1A, RN1B, RN1C, RN1D, RN2A, RN2B, RN2C, RN2D, RN3A, RN3B, RN3C, RN3D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
