File: projects/Redundant_Urgent_Data_Allocation_System/RUDAS_KID_LOW.brd (EAGLE design)
At the start: 160 x 100 mm, 13 parts, among them IC1 5M240ZT100, IC2 STM32F1_XL_DENSITY_LQFP144

Commit message: add connection
Parts:
- added C11, C12, C13, C14, C15, C16, C17, C18: (no value), rcl:C0805
- added CAN_GND, CAN_H, CAN_L, CAN_VCC, UART_GND, UART_RX, UART_TX, UART_VCC: TP, ORBiT-special:TP_SMD
- added U$2: ISO1050, ORBiT-IC-CAN-DRIVER:SOP8
- C1, C10, C2, C3, C4, C5, C6, C7, C8, C9: device rcl:C1210 -> rcl:C0805
- IC2: value STM32F1_XL_DENSITY_LQFP144 -> STM32F103VGT6
- moved IC1 44.0 mm to (59.3, 20.2), turned to 180 degrees
- moved IC2 40.4 mm to (21.6, 20.3), turned to 90 degrees
- moved U$1 11.6 mm to (42.0, 19.3), turned to 180 degrees
- moved C9 1.80 mm to (-16.5, 45.7)
- moved C10 1.80 mm to (-21.6, 45.7)
Connections:
- net IO_!BUSY! renamed FSMC_!NWAIT!
- net IO_R/!W! renamed FSMC_!WE!
- removed net IO_!CE!: U$1.55
- removed net IO_!OE!: U$1.48
- removed net VDD: IC2.108, IC2.121, IC2.131, IC2.144, IC2.17, IC2.39, IC2.52, IC2.62, IC2.72, IC2.84, IC2.95
- removed net VSS: IC2.107, IC2.120, IC2.130, IC2.143, IC2.16, IC2.38, IC2.51, IC2.61, IC2.71, IC2.83, IC2.94
- new net BOOT: IC2.138
- new net CAN_H: U$2.7
- new net CAN_L: U$2.6
- new net C_TCK: IC1.24
- new net C_TDI: IC1.23
- new net C_TDO: IC1.25
- new net C_TMS: IC1.22
- new net FSMC_!NE1!: IC2.123, U$1.55
- new net FSMC_!NOE!: IC2.118, U$1.48
- new net FSMC_!NWE!: IC2.119
- new net FSMC_!WAIT!: IC2.122
- new net GND1: U$2.4
- new net GND2: U$2.5
- new net STM32_CAN_RX: IC2.103, U$2.2
- new net STM32_CAN_TX: IC2.104, U$2.3
- new net STM32_I2C1_SCL: IC2.136
- new net STM32_I2C1_SDA: IC2.137
- new net STM32_SPI1_CS: IC2.40
- new net STM32_SPI1_MISO: IC2.42
- new net STM32_SPI1_MOSI: IC2.43
- new net STM32_SPI1_SCK: IC2.41
- new net STM32_UART1_RX: IC2.102, UART_RX.P$1
- new net STM32_UART1_TX: IC2.101, UART_TX.P$1
- new net STM32_UART2_RX: IC2.36
- new net STM32_UART2_TX: IC2.35
- new net S_GND: C11.2, C12.2, C13.2, C14.2, C15.2, C16.2, C17.2, C18.2, IC2.107, IC2.120, IC2.130, IC2.143, IC2.16, IC2.38, IC2.51, IC2.61, IC2.71, IC2.83, IC2.94
- new net S_OSC_IN: IC2.23
- new net S_OSC_OUT: IC2.24
- new net S_RST: IC2.25
- new net S_TCK: IC2.109
- new net S_TDI: IC2.110
- new net S_TDO: IC2.133
- new net S_TMS: IC2.105
- new net S_TRST: IC2.134
- new net S_VCC: C11.1, C12.1, C13.1, C14.1, C15.1, C16.1, C17.1, C18.1, IC2.108, IC2.121, IC2.131, IC2.144, IC2.17, IC2.39, IC2.52, IC2.62, IC2.72, IC2.84, IC2.95
- new net VCC1: U$2.1
- new net VCC2: U$2.8
- net FSMC_A0: now also IC2.10
- net FSMC_A1: now also IC2.11
- net FSMC_A2: now also IC2.12
- net FSMC_A3: now also IC2.13
- net FSMC_A4: now also IC2.14
- net FSMC_A5: now also IC2.15
- net FSMC_A6: now also IC2.50
- net FSMC_A7: now also IC2.53
- net FSMC_A8: now also IC2.54
- net FSMC_A9: now also IC2.55
- net FSMC_D0: now also IC2.85
- net FSMC_D1: now also IC2.86
- net FSMC_D2: now also IC2.114
- net FSMC_D3: now also IC2.115
- net FSMC_D4: now also IC2.58
- net FSMC_D5: now also IC2.59
- net FSMC_D6: now also IC2.60
- net FSMC_D7: now also IC2.63
Routing:
- net FSMC_A5: track 0.00 -> 3.80 mm
- net FSMC_A4: track 0.00 -> 3.80 mm
- net FSMC_A3: track 0.00 -> 3.80 mm
- net FSMC_A2: track 0.00 -> 3.80 mm
- net FSMC_A1: track 0.00 -> 3.80 mm
- net FSMC_A0: track 0.00 -> 3.80 mm
