File: projects/Redundant_Urgent_Data_Allocation_System/RUDAS_KID_designBox.sch (EAGLE design)
At the start: 46 parts, among them IC2 STM32F103VGT6, IC3 5M240ZT100

Commit message: add new part list
Parts:
- removed U$3: CONN-10PINR/A-10PIN, ORBIT-CONN HEADER-3M-2500 Series:CONN-10PINR/A-10PIN
- removed U$4: CONN-20PINR/A-20PIN, ORBIT-CONN HEADER-3M-2500 Series:CONN-20PINR/A-20PIN
- added J1: (no value), Wurth_Elektronik_Electromechanic_FPC_Connectors_&_Flat_Flexible_Cable_rev18c:686106183522
- added J2: (no value), Wurth_Elektronik_Electromechanic_FPC_Connectors_&_Flat_Flexible_Cable_rev18c:686108183422
Connections:
- net N$10 renamed 12V_GND
- net N$11 renamed +5V
- net N$12 renamed 3V_GND
- net N$5 renamed CAN_H_S
- net N$6 renamed CAN_L_S
- net N$7 renamed +12V
- net N$8 renamed 5V_GND
- net N$9 renamed +3V
- net CPLD_GND: now also J1.6; no longer U$3.PIN10, U$3.PIN6
- net CPLD_IO_VCC: now also J1.1; no longer U$3.PIN7, U$3.PIN8
- net C_TCK: now also J1.2; no longer U$3.PIN1
- net C_TDI: now also J1.5; no longer U$3.PIN5
- net C_TDO: now also J1.3; no longer U$3.PIN2
- net C_TMS: now also J1.4; no longer U$3.PIN3
- net LAN_CLK_N3: now also IC3.IO29
- net LAN_CLK_N4: now also IC3.IO19
- net LAN_CLK_N5: now also IC3.IO5
- net LAN_CLK_P3: now also IC3.IO28
- net LAN_CLK_P4: now also IC3.IO18
- net LAN_CLK_P5: now also IC3.IO4
- net LAN_N3: now also IC3.IO27
- net LAN_N4: now also IC3.IO17
- net LAN_N5: now also IC3.IO3
- net LAN_P3: now also IC3.IO26
- net LAN_P4: now also IC3.IO16
- net LAN_P5: now also IC3.IO2
- net S_GND: now also J2.8; no longer U$4.PIN12, U$4.PIN13, U$4.PIN14, U$4.PIN15, U$4.PIN16, U$4.PIN17, U$4.PIN18, U$4.PIN19, U$4.PIN20
- net S_RST: now also J2.7; no longer U$4.PIN9
- net S_TCK: now also J2.5; no longer U$4.PIN5
- net S_TDI: now also J2.3; no longer U$4.PIN3
- net S_TDO: now also J2.6; no longer U$4.PIN7
- net S_TMS: now also J2.4; no longer U$4.PIN4
- net S_TRST: now also J2.2; no longer U$4.PIN2
- net S_VCC: now also J2.1; no longer U$4.PIN1, U$4.PIN11
Other:
- moved on the sheet: R6, R7, R8, R9
