File: projects/Serial_Addressable_Thermometer/PLAN2 FINAL2.brd (EAGLE design)
At the start: 83.8 x 91.4 mm, 54 parts, among them J1 analog, J2 analog, J3 analog, J4 analog, J5 analog, J6 analog, J7 analog, J8 analog, J9 analog

Commit message: add part list and fix package problem
Parts:
- C1, C2, C3, C4, C5, C6, C7, C8, C9: device rcl:C1808 -> rcl:C0805
- moved C1 61.8 mm to (74.8, 20.2), turned to 0 degrees
- moved C7 61.8 mm to (74.8, 83.7), turned to 0 degrees
- moved J1 58.4 mm to (71.1, 5.08)
- moved J3 58.4 mm to (12.7, 5.08)
- moved J7 58.4 mm to (71.1, 68.6)
- moved J9 58.4 mm to (12.7, 68.6)
- moved MAINCON 58.4 mm to (71.1, 14.0)
- moved MAINCON2 58.4 mm to (12.7, 14.0)
- moved MAINCON6 58.4 mm to (71.1, 77.5)
- moved MAINCON8 58.4 mm to (12.7, 77.5)
- moved U$20 58.4 mm to (77.5, 77.5)
- moved U$21 58.4 mm to (71.1, 87.6)
- moved U$26 58.4 mm to (19.1, 77.5)
- moved U$27 58.4 mm to (12.7, 87.6)
- moved U$3 58.4 mm to (77.5, 14.0)
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Routing:
- net +5V1: track 72.4 -> 71.4 mm
- net +5V5: track 72.4 -> 71.4 mm
- net +5V4: track 72.4 -> 71.4 mm
- net +5V3: track 72.4 -> 71.4 mm
- net +5V8: track 72.4 -> 71.4 mm
- net +5V7: track 72.4 -> 71.4 mm
- net +5V6: track 72.4 -> 71.4 mm
- net +5V2: track 72.4 -> 71.4 mm
- net +5V: track 72.4 -> 71.4 mm
