File: projects/Serial_Addressable_Thermometer/plan2.brd (EAGLE design)
At the start: 25.4 x 27.9 mm, 6 parts, among them J1 analog

Commit message: add part list and fix package problem
Parts:
- C1: device rcl:C1808 -> rcl:C0805
- moved C1 3.43 mm to (16.4, 20.2), turned to 0 degrees
Routing:
- net +5V: track 72.4 -> 71.4 mm
Changed lines of the file:
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@@
 <attribute name="VALUE" x="12.7" y="17.155" size="1.27" layer="27" rot="R180" align="top-center"/>
 </element>
-<element name="C1" library="rcl" library_urn="urn:adsk.eagle:library:334" package="C1808" package3d_urn="urn:adsk.eagle:package:23689/2" value="47u" x="12.954" y="20.32" smashed="yes" rot="R180">
-<attribute name="NAME" x="17.854" y="20.652" size="1.27" layer="25" rot="R180"/>
-<attribute name="SPICEPREFIX" value="C" x="12.954" y="20.32" size="1.778" layer="27" rot="R180" display="off"/>
-<attribute name="VALUE" x="9.98" y="20.622" size="1.27" layer="27" rot="R180"/>
+<element name="C1" library="rcl" library_urn="urn:adsk.eagle:library:334" package="C0805" package3d_urn="urn:adsk.eagle:package:23617/2" value="47u" x="16.383" y="20.193" smashed="yes">
+<attribute name="NAME" x="11.483" y="19.861" size="1.27" layer="25"/>
+<attribute name="SPICEPREFIX" value="C" x="16.383" y="20.193" size="1.778" layer="27" display="off"/>
+<attribute name="VALUE" x="19.357" y="19.891" size="1.27" layer="27"/>
 </element>
 <element name="U$2" library="ORBiT-con-JST" package="JST_ZH_4PIN" value="IIC1" x="6.35" y="13.97" smashed="yes" rot="R270">
@@
 <wire x1="5.8646" y1="14.7546" x2="7.62" y2="16.51" width="0.508" layer="16"/>
 <contactref element="C1" pad="1"/>
-<wire x1="19.05" y1="17.78" x2="16.51" y2="20.32" width="0.508" layer="1"/>
-<wire x1="16.51" y1="20.32" x2="14.904" y2="20.32" width="0.508" layer="1"/>
-<wire x1="19.05" y1="15.47" x2="19.05" y2="17.78" width="0.508" layer="1"/>
-<wire x1="16.9917" y1="18.2323" x2="14.904" y2="20.32" width="0.254" layer="1"/>
-<wire x1="16.9917" y1="12.75726875" x2="16.9917" y2="18.2323" width="0.254" layer="1"/>
-<wire x1="14.904" y1="20.32" x2="15.24" y2="20.656" width="0.508" layer="1"/>
-<wire x1="15.24" y1="20.656" x2="15.24" y2="22.72" width="0.508" layer="1"/>
+<wire x1="19.05" y1="15.47" x2="19.05" y2="16.51" width="0.508" layer="1"/>
+<wire x1="19.05" y1="16.51" x2="16.5234" y2="19.0366" width="0.508" layer="1"/>
+<wire x1="16.5234" y1="19.0366" x2="16.5146625" y2="19.0366" width="0.508" layer="1"/>
+<wire x1="16.5146625" y1="19.0366" x2="15.60423125" y2="19.94703125" width="0.508" layer="1"/>
+<wire x1="15.60423125" y1="19.94703125" x2="15.433" y2="20.1182625" width="0.508" layer="1"/>
+<wire x1="15.433" y1="20.1182625" x2="15.433" y2="20.193" width="0.508" layer="1"/>
+<wire x1="15.433" y1="19.907" x2="15.2" y2="20.14" width="0.508" layer="1"/>
+<wire x1="15.2" y1="22.68" x2="15.2" y2="20.14" width="0.508" layer="1"/>
+<wire x1="15.433" y1="19.907" x2="15.433" y2="20.193" width="0.508" layer="1"/>
+<wire x1="16.9917" y1="17.78" x2="15.433" y2="19.3387" width="0.254" layer="1"/>
+<wire x1="15.433" y1="19.3387" x2="15.433" y2="20.193" width="0.254" layer="1"/>
+<wire x1="16.9917" y1="12.75726875" x2="16.9917" y2="17.78" width="0.254" layer="1"/>
 </signal>
 <signal name="N$1">
