File: projects/Serial_Addressable_Thermometer/sensorboard.brd (EAGLE design)
At the start: 36.8 x 20 mm, 4 parts

Commit message: add part list and fix package problem
Parts:
- R1, R9: device rcl:R1210 -> rcl:R0805
- moved OUT 10.2 mm to (21.6, 10.2)
- moved R9 5.12 mm to (13.7, 5.71)
- moved R1 5.08 mm to (13.7, 14.0)
Routing:
- net N$1: track 100.0 -> 0.00 mm
- net S$1: track 20.0 -> 0.00 mm
- net +5V: track 31.8 -> 16.4 mm
- net AGND: track 30.5 -> 15.4 mm
- net AD5: track 22.3 -> 12.1 mm
- net AD8: track 22.3 -> 12.1 mm
- net AD6: track 22.3 -> 12.1 mm
- net AD4: track 22.3 -> 12.1 mm
- net AD3: track 22.3 -> 12.1 mm
- net AD2: track 22.3 -> 12.1 mm
- net AD7: track 22.3 -> 12.1 mm
- net ADB: track 15.8 -> 11.8 mm
Other:
- board size 36.8 x 20 mm -> 26.6 x 19.7 mm
